Commit message: 暂存一版

File: ros_ws/src/eli_cs_robot_description/urdf/cs.ros2_control.xacro (robot description, xacro)
@@ -21,5 +21,5 @@
     script_command_port:=50004
     trajectory_port:=50003
-    robot_receive_timeout:=0.2
+    robot_receive_timeout:=0.5
     ">
     <ros2_control name="${name}" type="system">

File: ros_ws/src/eli_cs_robot_description/urdf/cs.urdf.xacro (robot description, xacro)
@@ -5,4 +5,5 @@
    <!-- import main macro -->
    <xacro:include filename="$(find eli_cs_robot_description)/urdf/cs_macro.xacro"/>
+   <xacro:include filename="$(find eli_cs_robot_description)/urdf/cs_macro_terminal.xacro"/>
    <!-- possible 'cs_type' values: cs63, cs66, cs66a, cs68, cs612, cs616, cs618f, cs620, cs625, ls65 -->
    <!-- the default value should raise an error in case this was called without defining the type -->
@@ -45,4 +46,13 @@
    <!-- initial position for simulations (Fake Hardware, Gazebo, Ignition) -->
    <xacro:arg name="initial_positions_file" default="$(find eli_cs_robot_description)/config/initial_positions.yaml"/>
+   <!-- 同一末端装配供真机、MoveIt、导纳和模型预览共同使用。 -->
+   <xacro:arg name="attach_terminal" default="true"/>
+   <xacro:arg name="terminal_mesh_base" default="package://eli_cs_robot_description/meshes/terminal"/>
+   <xacro:arg name="terminal_x" default="0.0"/>
+   <xacro:arg name="terminal_y" default="0.0"/>
+   <xacro:arg name="terminal_z" default="0.0"/>
+   <xacro:arg name="terminal_roll" default="0.0"/>
+   <xacro:arg name="terminal_pitch" default="0.0"/>
+   <xacro:arg name="terminal_yaw" default="-1.5707963267948966"/>
    <!-- convert to property to use substitution in function -->
    <xacro:property name="initial_positions_file" default="$(arg initial_positions_file)"/>
@@ -87,4 +97,10 @@
      <origin xyz="0 0 0" rpy="0 0 0" />          <!-- position robot in the world -->
    </xacro:cs_robot>
+   <xacro:if value="$(arg attach_terminal)">
+     <xacro:cs_terminal tf_prefix="$(arg tf_prefix)"
+       mesh_base="$(arg terminal_mesh_base)"
+       x="$(arg terminal_x)" y="$(arg terminal_y)" z="$(arg terminal_z)"
+       roll="$(arg terminal_roll)" pitch="$(arg terminal_pitch)" yaw="$(arg terminal_yaw)"/>
+   </xacro:if>
    <xacro:if value="$(arg sim_gazebo)">
     <!-- Gazebo plugins -->

File: ros_ws/src/eli_cs_robot_moveit_config/srdf/cs.srdf.xacro (robot description, xacro)
@@ -5,5 +5,6 @@
   <!-- parameters -->
   <xacro:arg name="prefix" default="" />
+  <xacro:arg name="attach_terminal" default="true"/>
   <xacro:include filename="$(find eli_cs_robot_moveit_config)/srdf/cs_macro.srdf.xacro"/>
-  <xacro:cs_srdf name="$(arg name)" prefix="$(arg prefix)"/>
+  <xacro:cs_srdf name="$(arg name)" prefix="$(arg prefix)" attach_terminal="$(arg attach_terminal)"/>
 </robot>

File: ros_ws/src/eli_cs_robot_moveit_config/srdf/cs_macro.srdf.xacro (robot description, xacro)
@@ -5,5 +5,5 @@
     A URDF file must exist for this robot as well, where the joints and the links that are referenced are defined
 -->
-  <xacro:macro name="cs_srdf" params="name prefix">
+  <xacro:macro name="cs_srdf" params="name prefix attach_terminal:=true">
     <!--GROUPS - Representation of a set of joints and links. This can be useful for specifying DOF to plan for, defining arms, end effectors, etc-->
     <!--LINKS - When a link is specified, the parent joint of that link (if it exists) is automatically included-->
@@ -41,4 +41,13 @@
     <!--END EFFECTOR - Purpose - Represent information about an end effector.-->
     <!--VIRTUAL JOINT - Purpose - this element defines a virtual joint between a robot link and an external frame of reference (considered fixed with respect to the robot)-->
+    <!-- 同一刚性装配内部和腕部安装面允许接触；其余机械臂碰撞检查保留。 -->
+    <xacro:if value="${attach_terminal}">
+      <disable_collisions link1="${prefix}terminal_base_link" link2="${prefix}terminal_link_1" reason="Adjacent"/>
+      <disable_collisions link1="${prefix}terminal_base_link" link2="${prefix}terminal_link_2" reason="Adjacent"/>
+      <disable_collisions link1="${prefix}terminal_link_1" link2="${prefix}terminal_link_2" reason="RigidAssembly"/>
+      <disable_collisions link1="${prefix}wrist_3_link" link2="${prefix}terminal_base_link" reason="Adjacent"/>
+      <disable_collisions link1="${prefix}wrist_3_link" link2="${prefix}terminal_link_1" reason="RigidAssembly"/>
+      <disable_collisions link1="${prefix}wrist_3_link" link2="${prefix}terminal_link_2" reason="RigidAssembly"/>
+    </xacro:if>
     <!--DISABLE COLLISIONS - By default it is assumed that any link of the robot could potentially come into collision with any other link in the robot. This tag disables collision checking between a specified pair of links. -->
     <disable_collisions link1="${prefix}base_link" link2="${prefix}base_link_inertia" reason="Adjacent" />
